File: project/load_v2/relay.sch (KiCad schematic (older format))
At the start: 9 parts, among them P11 relay, P12 N, P13 S, Q4 2n222, Q5 2n222

Commit message: 3fet
Changed lines of the file:
@@
 $Descr A4 11693 8268
 encoding utf-8
-Sheet 2 2
+Sheet 2 3
 Title ""
 Date ""
@@
 $EndComp
 $Comp
-L +12V #PWR54
+L +12V #PWR051
 U 1 1 584873BE
 P 1750 1400
-F 0 "#PWR54" H 1750 1250 50  0001 C CNN
+F 0 "#PWR051" H 1750 1250 50  0001 C CNN
 F 1 "+12V" H 1750 1540 50  0000 C CNN
 F 2 "" H 1750 1400 50  0000 C CNN
@@
 $EndComp
 $Comp
-L GND #PWR55
+L GND #PWR052
 U 1 1 584873D4
 P 1750 1950
-F 0 "#PWR55" H 1750 1700 50  0001 C CNN
+F 0 "#PWR052" H 1750 1700 50  0001 C CNN
 F 1 "GND" H 1750 1800 50  0000 C CNN
 F 2 "" H 1750 1950 50  0000 C CNN
@@
 $EndComp
 $Comp
-L GND #PWR57
+L GND #PWR053
 U 1 1 5848974B
 P 2400 2650
-F 0 "#PWR57" H 2400 2400 50  0001 C CNN
+F 0 "#PWR053" H 2400 2400 50  0001 C CNN
 F 1 "GND" H 2400 2500 50  0000 C CNN
 F 2 "" H 2400 2650 50  0000 C CNN
@@
 $EndComp
 $Comp
-L GND #PWR59
+L GND #PWR054
 U 1 1 5848976B
 P 3500 3150
-F 0 "#PWR59" H 3500 2900 50  0001 C CNN
+F 0 "#PWR054" H 3500 2900 50  0001 C CNN
 F 1 "GND" H 3500 3000 50  0000 C CNN
 F 2 "" H 3500 3150 50  0000 C CNN
@@
 $EndComp
 $Comp
-L +12V #PWR56
+L +12V #PWR055
 U 1 1 5848988A
 P 2400 1400
-F 0 "#PWR56" H 2400 1250 50  0001 C CNN
+F 0 "#PWR055" H 2400 1250 50  0001 C CNN
 F 1 "+12V" H 2400 1540 50  0000 C CNN
 F 2 "" H 2400 1400 50  0000 C CNN
@@
 $EndComp
 $Comp
-L +12V #PWR58
+L +12V #PWR056
 U 1 1 584898AA
 P 3500 1400
-F 0 "#PWR58" H 3500 1250 50  0001 C CNN
+F 0 "#PWR056" H 3500 1250 50  0001 C CNN
 F 1 "+12V" H 3500 1540 50  0000 C CNN
 F 2 "" H 3500 1400 50  0000 C CNN
@@
 	3500 1400 3500 1450
 Wire Wire Line
-	2400 2050 2400 2100
-Wire Wire Line
-	2400 2100 2400 2200
-Wire Wire Line
-	3500 2050 3500 2100
-Wire Wire Line
-	3500 2100 3500 2700
+	2400 2050 2400 2200
+Wire Wire Line
+	3500 2050 3500 2700
 Wire Wire Line
 	3500 3100 3500 3150
