File: project/load_v2/v2.sch (KiCad schematic (older format))
At the start: 118 parts, among them IC1 ATMEGA328-P, P1 12VAC, P10 relay, P2 NGUON, P3 SAC, P4 12N60C, P5 CONN_01X02, P6 button, P7 UART, P8 FAN, P9 7-seg, Q1 Q_NPN_BCE, Q2 Q_NPN_BCE, Q3 Q_NPN_BCE, SW1 reset, U1 LM7812CT, U2 LM7805CT, U3 ICL7660, U4 TL431, U5 LM324N, U6 LM324N, U7 LM7812CT, Y1 16MHz

Commit message: 3fet
Connections:
- net set_I: now reaches C17.2, R21.1, U5.12 (+)
