File: project/load_v3/v3.sch (KiCad schematic (older format))
At the start: 118 parts, among them IC1 ATMEGA328-P, P1 12VAC, P10 relay, P2 NGUON, P3 SAC, P4 12N60C, P5 CONN_01X02, P6 button, P7 UART, P8 FAN, P9 7-seg, Q1 Q_NPN_BCE, Q2 Q_NPN_BCE, Q3 Q_NPN_BCE, SW1 reset, U1 LM7812CT, U2 LM7805CT, U3 ICL7660, U4 TL431, U5 LM324N, U6 LM324N, U7 LM7812CT, Y1 16MHz

Commit message: a
Parts:
- removed C18: 100nF, Capacitors_THT:C_Rect_L7_W2_P5, symbol C
- removed C19: 22nF, Capacitors_THT:C_Disc_D3_P2.5, symbol C
- removed C21: 100nF, Capacitors_THT:C_Disc_D3_P2.5, symbol C
- removed D8: 5.1V, Diodes_THT:Diode_DO-35_SOD27_Horizontal_RM10, symbol ZENER
- removed P4: 12N60C, Connectors_Phoenix:PhoenixContact_MCV-G_05x5.08mm_Vertical, symbol CONN_01X05
- removed R22: 470R, Resistors_THT:Resistor_Horizontal_RM7mm, symbol R
- removed R23: 1k, Resistors_THT:Resistor_Horizontal_RM7mm, symbol R
- removed R28: 330R, Resistors_THT:Resistor_Horizontal_RM7mm, symbol R
- removed R29: 10k, Resistors_THT:Resistor_Horizontal_RM15mm, symbol R
- removed R30: 180k, Resistors_THT:Resistor_Horizontal_RM15mm, symbol R
- removed R46: 10k, Resistors_THT:Resistor_Horizontal_RM7mm, symbol R
- removed R47, R48, R49, R50, R51, R52, R53, R54, R55, R56, R57: 0R, Wire_Connections_Bridges:WireConnection_0.80mmDrill, symbol R
- removed RV2: 20k, Potentiometers:Potentiometer_Bourns_3296W_3-8Zoll_Inline_ScrewUp, symbol POT-RESCUE-v2
- removed U6: LM324N, Housings_DIP:DIP-14_W7.62mm_LongPads, symbol LM324N
- added D12, D13: 4001, Diodes_THT:Diode_DO-35_SOD27_Horizontal_RM10, symbol D_Small
- added D14, D8: Led_Small, LEDs:LED-3MM, symbol Led_Small
- added P11: G, Connectors:XH2.54-3P, symbol CONN_01X03
- added P12: N, Connectors_Phoenix:PhoenixContact_MCV-G_02x5.08mm_Vertical, symbol CONN_01X02
- added P13: S, Connectors_Phoenix:PhoenixContact_MCV-G_02x5.08mm_Vertical, symbol CONN_01X02
- added P4: DS, Connectors_Phoenix:PhoenixContact_MCV-G_02x5.08mm_Vertical, symbol CONN_01X02
- added Q4, Q5: 2n222, TO_SOT_Packages_THT:TO-92_Molded_Wide_Oval_Reverse, symbol Q_NPN_BCE
- added RL1: onN, Relays_THT:Relay_SPDT_OMRON-G5Q, symbol G5Q-1
- added RL2: onS, Relays_THT:Relay_SPDT_OMRON-G5Q, symbol G5Q-1
- added VR3: 14D180V, Varistors:RV_Disc_D15.5_W3.9_P7.5, symbol VR
- C1: footprint Capacitors_THT:C_Radial_D5_L6_P2.5 -> Capacitors_THT:C_Radial_D8_L11.5_P3.5
- D1: footprint Diodes_THT:Diode_Bridge_18.5x5.5 -> Diodes_THT:Diode_Bridge_KBP206
- P10: value relay -> overheat
- Q1, Q2, Q3, U4: footprint TO_SOT_Packages_THT:TO-92_Molded_Narrow -> TO_SOT_Packages_THT:TO-92_Molded_Wide_Oval_Reverse
- R41, R45: value 10k -> 470R; footprint Resistors_THT:Resistor_Horizontal_RM7mm -> Resistors_SMD:R_0805_HandSoldering
- VR1, VR2: value 14D470K -> 14D180V
- Y1: footprint Crystals:Crystal_HC52-U_Vertical -> Crystals:Crystal_HC50-U_Vertical
Connections:
- net +12V: now also P11.3 (P3); no longer D7.1 (K), P8.1 (P1), R41.2, R45.2
- net +5V: now also C10.2, IC1.7 (VCC), R7.1, U3.8 (VCC)
- net -5V: now also P11.1 (P1); no longer U5.11 (V-)
- net 12V2: no longer U5.4 (V+)
- net 12Vrelay: now also D7.1 (K), P10.4 (P4), P8.1 (P1), D12.1 (K), D13.1 (K), RL1.5, RL2.5; no longer P10.1 (P1)
- net D: now also P4.1 (P1)
- net G: now also C17.2, R21.1, P11.2 (P2)
- net GND: now also P10.1 (P1), Q3.3 (E), U5.5 (+), D14.1 (K), D8.1 (K), Q4.3 (E), Q5.3 (E); no longer P10.4 (P4)
- net S: now also R26.1, P4.2 (P2)
- net onN: now also Q4.1 (B); no longer P10.2 (P2)
- net onS: now also Q5.1 (B); no longer P10.3 (P3)
- net at D1.2, P1.1 (P1): now also VR3.2
- net at D1.4, P1.2 (P2): now also VR3.1
- net ok: now reaches IC1.27 ((PCINT12/SDA/ADC4)PC4)
- net ok: now also R41.2
- net fail: now reaches IC1.28 ((PCINT13/SCL/ADC5)PC5)
- net fail: now also R45.2
- net at U5.6 (-): now also R34.1, R35.2; no longer U5.7
- net at D11.1 (K), R31.1: now also U5.8, U5.9 (-); no longer U5.1, U5.2 (-)
- net at D9.1 (K), R24.1, R25.2: now also U5.14; no longer U5.8
- net at D10.1 (K), R36.1, R37.2: now also U5.1
- net at R26.2: now also U5.12 (+); no longer U5.10 (+)
- net at R25.1, R27.2: now also U5.13 (-); no longer U5.9 (-)
- net at R32.1, R33.2: now also U5.10 (+); no longer U5.3 (+)
- net at R34.2, R38.1: now also U5.7
- net at R38.2: now also U5.2 (-)
- net at R37.1, R39.2: now also U5.3 (+)
- net at R45.1: now also D14.2 (A)
- net at R40.1: now also Q1.1 (B), Q2.1 (B)
- net at R44.1: now also Q3.1 (B)
- net off: now reaches R40.2
- net off: now also P10.3 (P3)
- net onFan: now reaches R44.2
- net onFan: now also P10.2 (P2); no longer Q3.1 (B)
- net THa: no longer names the net of R41.1
- net THa: now also D8.2 (A)
- removed net set_I: C17.2, R21.1, U5.12 (+)
- new net: D12.2 (A), Q4.2 (C), RL1.1
- new net: P12.2 (P2), RL1.2
- new net: P12.1 (P1), RL1.3
- new net: D13.2 (A), Q5.2 (C), RL2.1
- new net: P13.1 (P1), RL2.3
- new net: P13.2 (P2), RL2.2
Other:
- note added: "0-2.5V ->"
- note added: "5V Vref"
- note added: "<- 0-0.5V"
- note removed: "0-0.5V"
- note removed: "40*C-52.6k"
- note removed: "90*C-10k"
- note removed: "NTC-MF58 100K 3950 5%"
- note removed: "Sau mạch lọc"
- moved on the sheet: C16, C17, C20, C22, C23, D10, D11, D5, D7, D9, P8, Q1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

Commit message: a
Parts:
- removed R42: 1k, Resistors_THT:Resistor_Horizontal_RM7mm, symbol R
- added R? (x2): 10k, Resistors_THT:Resistor_Horizontal_RM7mm, symbol R
- added U10, U9: PC817, DIP-4, symbol PC817
- P12: value N -> opto_auto; footprint Connectors_Phoenix:PhoenixContact_MCV-G_02x5.08mm_Vertical -> (none)
- P13: value S -> opto_start; footprint Connectors_Phoenix:PhoenixContact_MCV-G_02x5.08mm_Vertical -> (none)
- RL1, RL2: footprint Relays_THT:Relay_SPDT_OMRON-G5Q -> Relays_THT:Relay_SANYOU_SRD_Series_Form_C
Connections:
- net onS is gone; now on net onN: Q2.2 (C), Q5.1 (B), R43.1
- net +5V: no longer R19.1
- net D: now also RL2.1; no longer P3.2 (P2)
- net GND: now also D6.1 (K), U10.2, U9.2
- net N+: now also RL1.1; no longer D5.2 (A)
- net start: now also IC1.14 ((PCINT0/CLKO/ICP1)PB0), R19.1, R?.2
- net at D12.2 (A), Q4.2 (C): now also RL1.2; no longer RL1.1
- net at P12.2 (P2): now also U9.4; no longer RL1.2
- net at P12.1 (P1): now also U9.3; no longer RL1.3
- net at D13.2 (A), Q5.2 (C): now also RL2.2; no longer RL2.1
- net at P13.1 (P1): now also U10.3; no longer RL2.3
- net at P13.2 (P2): now also U10.4; no longer RL2.2
- net led: no longer names the net of IC1.13 ((PCINT23/AIN1)PD7)
- net led: now also R?.2; no longer D6.1 (K)
- new net S+: P3.2 (P2), RL2.3
- new net opto_auto: R?.1, U9.1
- new net opto_start: R?.1, U10.1
- new net rN+: D5.2 (A), RL1.3
Other:
- note added: "hold start 1s to enter auto mode"
- moved on the sheet: D6, R19

Commit message: a
Parts:
- removed P12: opto_auto, symbol CONN_01X02
- removed P13: opto_start, symbol CONN_01X02
- added P12: opto, Connectors:XH2.54-4P, symbol CONN_01X04
- U10, U9: footprint DIP-4 -> Housings_DIP:DIP-4_W7.62mm_LongPads
- gave numbers to parts that had none: 2
Connections:
- net at U9.3: now also P12.3 (P3)
- net at U9.4: now also P12.4 (P4)
- net at U10.3: now also P12.1 (P1)
- net at U10.4: now also P12.2 (P2)

Commit message: a
Parts:
- removed D6: Led_Small, LEDs:LED-3MM, symbol Led_Small
- removed VR2: 14D180V, Varistors:RV_Disc_D15.5_W3.9_P7.5, symbol VR
- added D15, D16: Led_Small, LEDs:LED-3MM, symbol Led_Small
- added P13: tac_auto, Connectors:XH2.54-2P, symbol CONN_01X02
- added R47: 470R, Resistors_SMD:R_0805_HandSoldering, symbol R
- R19: footprint Resistors_THT:Resistor_Horizontal_RM7mm -> Resistors_SMD:R_0805_HandSoldering
- R42, R46: value 10k -> 1k
Connections:
- net GND: now also VR1.2, D15.1 (K), D16.1 (K), P13.2 (P2)
- net S-: no longer VR1.2
- net opto_auto: now also U10.1; no longer U9.1
- net opto_start: now also U9.1; no longer U10.1
- net start: now also P13.1 (P1); no longer IC1.14 ((PCINT0/CLKO/ICP1)PB0), R19.1, R42.2
- net l_auto: now reaches IC1.13 ((PCINT23/AIN1)PD7), R46.2
- net l_auto: now also R19.2
- net at D11.1 (K), R31.1: now also U5.13 (-), U5.14; no longer U5.8, U5.9 (-)
- net at D9.1 (K), R24.1, R25.2: now also U5.1; no longer U5.14
- net at D10.1 (K), R36.1, R37.2: now also U5.8; no longer U5.1
- net at R38.2: now also U5.9 (-); no longer U5.2 (-)
- net at R37.1, R39.2: now also U5.10 (+); no longer U5.3 (+)
- net at R26.2: now also U5.3 (+); no longer U5.12 (+)
- net at R25.1, R27.2: now also U5.2 (-); no longer U5.13 (-)
- net at R32.1, R33.2: now also U5.12 (+); no longer U5.10 (+)
- new net: D15.2 (A), R19.1
- new net: D16.2 (A), R47.1
- new net l_start: IC1.14 ((PCINT0/CLKO/ICP1)PB0), R42.2, R47.2
Other:
- note added: "Us = Un - Udiode"
- moved on the sheet: D14, D2, D3, D4, D8, R4, R41, R45, R5, R6, VR1
