File: project/load_v3/v3.sch (KiCad schematic (older format))
At the start: 111 parts, among them IC1 ATMEGA328-P, P1 12VAC, P10 overheat, P11 G, P12 opto, P13 tac_auto, P2 NGUON, P3 SAC, P4 DS, P5 CONN_01X02, P6 button, P7 UART, P8 FAN, P9 7-seg, Q1 Q_NPN_BCE, Q2 Q_NPN_BCE, Q3 Q_NPN_BCE, Q4 2n222, Q5 2n222, SW1 reset, U1 LM7812CT, U10 PC817, U2 LM7805CT, U3 ICL7660, U4 TL431, U5 LM324N, U7 LM7812CT, U9 PC817, Y1 16MHz

Commit message: a
Connections:
- net 12V2 is gone; now on net +12V: R1.2
- net senIN: now also IC1.24 ((PCINT9/ADC1)PC1); no longer IC1.23 ((PCINT8/ADC0)PC0)
- net senIS: now also IC1.25 ((PCINT10/ADC2)PC2); no longer IC1.26 ((PCINT11/ADC3)PC3), R36.2
- net senUN: now also IC1.26 ((PCINT11/ADC3)PC3); no longer IC1.25 ((PCINT10/ADC2)PC2)
- net senUS: now also IC1.23 ((PCINT8/ADC0)PC0); no longer IC1.24 ((PCINT9/ADC1)PC1)
Other:
- moved on the sheet: C16, C17, C20, C22, C23, D10, D11, D12, D13, D14, D15, D16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
