File: project/load_v3/v3.sch (KiCad schematic (older format))
At the start: 111 parts, among them IC1 ATMEGA328-P, P1 12VAC, P10 overheat, P11 G, P12 opto, P13 tac_auto, P2 NGUON, P3 SAC, P4 DS, P5 CONN_01X02, P6 button, P7 UART, P8 FAN, P9 7-seg, Q1 Q_NPN_BCE, Q2 Q_NPN_BCE, Q3 Q_NPN_BCE, Q4 2n222, Q5 2n222, SW1 reset, U1 LM7812CT, U10 PC817, U2 LM7805CT, U3 ICL7660, U4 TL431, U5 LM324N, U7 LM7812CT, U9 PC817, Y1 16MHz

Commit message: chager
Connections:
- net GND: now also D4.2 (A); no longer D4.1 (K)
- net at R6.1: now also D4.1 (K); no longer D4.2 (A)
Other:
- moved on the sheet: D4
