File: project/load_v3/3FET.sch (KiCad schematic (older format))
At the start: 24 parts, among them P14 IN, P15 OUT, Q6 Q_NMOS_GDS, Q7 Q_NMOS_GDS, Q8 Q_NMOS_GDS, U8 LM324

Commit message: a
Parts:
- removed C24: 22nF, symbol C
- removed P14: IN, symbol CONN_01X05
- removed P15: OUT, symbol CONN_01X03
- removed Q8: Q_NMOS_GDS, symbol Q_NMOS_GDS
- removed R63: 0.1R, symbol R
- removed R65, R66, R70: 1k, symbol R
- removed R67, R68: 8.2k, symbol R
- removed R69: 470R, symbol R
- removed R71: 0.5R, symbol R
- removed TH1: THERMISTOR, symbol THERMISTOR
- removed U8: LM324, symbol LM324
- added P14: pwr, Connectors_Phoenix:PhoenixContact_MCV-G_02x5.08mm_Vertical, symbol CONN_01X02
- added P16: g, Connectors:XH2.54-3P, symbol CONN_01X03
- added R29, R30: 10k, Resistors_THT:Resistor_Horizontal_RM7mm, symbol R
- added U8: LM358, Housings_DIP:DIP-8_W7.62mm_LongPads, symbol LM358
- C14, C8: footprint (none) -> Capacitors_THT:C_Disc_D3_P2.5
- Q6, Q7: footprint (none) -> TO_SOT_Packages_THT:TO-247_Vertical_Neutral123
- R58, R59, R61, R62: footprint (none) -> Resistors_THT:Resistor_Horizontal_RM7mm
- R60, R64: footprint (none) -> Resistors_THT:Resistor_Vertical_RM7.5mm
Connections:
- net D: now also Q6.2 (D), Q7.2 (D), P14.1 (P1)
- net G: now also P16.2 (P2), U8.3 (+), U8.5 (+)
- net at Q6.3 (S), R59.1, R60.1: now also R29.1
- net at Q7.3 (S), R62.1, R64.1: now also R30.1
- net at Q6.1 (G), R58.1: now also R29.2
- net at C8.1, R58.2: now also U8.1
- net at Q7.1 (G), R61.1: now also R30.2
- net at C14.1, R61.2: now also U8.7
- net at C8.2, R59.2: now also U8.2 (-)
- net at C14.2, R62.2: now also U8.6 (-)
- net GNDA renamed S
- net S: now also P14.2 (P2)
- new net +12V: P16.3 (P3), U8.8 (V+)
- new net -5V: P16.1 (P1), U8.4 (V-)
Other:
- note added: "max = 5A\nUg = 5*0.5 = 2.5V"
- note removed: "S->GND"
- moved on the sheet: C14, C8, Q6, Q7, R58, R59, R60, R61, R62, R64

Commit message: a
Connections:
- net +12V: now also P16.1 (P1); no longer P16.3 (P3)
- net -5V: now also P16.3 (P3); no longer P16.1 (P1)
Changed lines of the file:
@@
 F 3 "" H 2400 4100 50  0000 C CNN
 	1    2400 4100
-	-1   0    0    1
+	-1   0    0    -1
 $EndComp
 $Comp
-L +12V #PWR54
+L +12V #PWR052
 U 1 1 5885AAC5
 P 2700 4000
-F 0 "#PWR54" H 2700 3850 50  0001 C CNN
+F 0 "#PWR052" H 2700 3850 50  0001 C CNN
 F 1 "+12V" H 2700 4140 50  0000 C CNN
 F 2 "" H 2700 4000 50  0000 C CNN
@@
 $EndComp
 $Comp
-L -5V #PWR55
+L -5V #PWR56
 U 1 1 5885AB09
 P 2700 4200
-F 0 "#PWR55" H 2700 4300 50  0001 C CNN
+F 0 "#PWR56" H 2700 4300 50  0001 C CNN
 F 1 "-5V" H 2700 4350 50  0000 C CNN
 F 2 "" H 2700 4200 50  0000 C CNN
@@
 $EndComp
 $Comp
-L +12V #PWR56
+L +12V #PWR053
 U 1 1 5885AD5B
 P 3650 3500
-F 0 "#PWR56" H 3650 3350 50  0001 C CNN
+F 0 "#PWR053" H 3650 3350 50  0001 C CNN
 F 1 "+12V" H 3650 3640 50  0000 C CNN
 F 2 "" H 3650 3500 50  0000 C CNN
@@
 $EndComp
 $Comp
-L -5V #PWR57
+L -5V #PWR58
 U 1 1 5885AF06
 P 3650 4500
-F 0 "#PWR57" H 3650 4600 50  0001 C CNN
+F 0 "#PWR58" H 3650 4600 50  0001 C CNN
 F 1 "-5V" H 3650 4650 50  0000 C CNN
 F 2 "" H 3650 4500 50  0000 C CNN
