File: project/load_v3/overheat.sch (KiCad schematic (older format))
At the start: 7 parts, among them P15 overheat, U9 LM324N

Commit message: a
Parts:
- removed U9: LM324N, Housings_DIP:DIP-14_W7.62mm_LongPads, symbol LM324N
- added U6: LM358, Housings_DIP:DIP-8_W7.62mm_LongPads, symbol LM358
Connections:
- net 12Vrelay: now also U6.8 (V+)
- net GND: now also U6.4 (V-)
- net off: now also U6.1
- net onFan: now also U6.7
- net at R28.1, TH2.1: now also U6.2 (-), U6.6 (-)
- net at R22.1, R23.2: now also U6.3 (+)
- net at RV3.2: now also U6.5 (+)
Changed lines of the file:
@@
 $EndDescr
 $Comp
-L LM324N U9
-U 1 1 5872C08F
-P 5550 3200
-F 0 "U9" H 5600 3400 50  0000 C CNN
-F 1 "LM324N" H 5700 3000 50  0000 C CNN
-F 2 "Housings_DIP:DIP-14_W7.62mm_LongPads" H 5500 3300 50  0001 C CNN
-F 3 "" H 5600 3400 50  0000 C CNN
-	1    5550 3200
-	-1   0    0    1
-$EndComp
-$Comp
-L LM324N U9
-U 2 1 5872C096
-P 5550 4500
-F 0 "U9" H 5600 4700 50  0000 C CNN
-F 1 "LM324N" H 5700 4300 50  0000 C CNN
-F 2 "Housings_DIP:DIP-14_W7.62mm_LongPads" H 5500 4600 50  0001 C CNN
-F 3 "" H 5600 4700 50  0000 C CNN
-	2    5550 4500
-	-1   0    0    1
-$EndComp
-$Comp
-L GND #PWR047
+L GND #PWR52
 U 1 1 5872C09D
 P 5650 4100
-F 0 "#PWR047" H 5650 3850 50  0001 C CNN
+F 0 "#PWR52" H 5650 3850 50  0001 C CNN
 F 1 "GND" H 5650 3950 50  0000 C CNN
 F 2 "" H 5650 4100 50  0000 C CNN
@@
 $EndComp
 $Comp
-L GND #PWR048
+L GND #PWR54
 U 1 1 5872C0AA
 P 6400 3750
-F 0 "#PWR048" H 6400 3500 50  0001 C CNN
+F 0 "#PWR54" H 6400 3500 50  0001 C CNN
 F 1 "GND" H 6400 3600 50  0000 C CNN
 F 2 "" H 6400 3750 50  0000 C CNN
@@
 $EndComp
 $Comp
-L GND #PWR049
+L GND #PWR53
 U 1 1 5872C0C7
 P 6100 4850
-F 0 "#PWR049" H 6100 4600 50  0001 C CNN
+F 0 "#PWR53" H 6100 4600 50  0001 C CNN
 F 1 "GND" H 6100 4700 50  0000 C CNN
 F 2 "" H 6100 4850 50  0000 C CNN
@@
 $EndComp
 $Comp
-L GND #PWR050
+L GND #PWR51
 U 1 1 5872CED6
 P 4700 2850
-F 0 "#PWR050" H 4700 2600 50  0001 C CNN
+F 0 "#PWR51" H 4700 2600 50  0001 C CNN
 F 1 "GND" H 4700 2700 50  0000 C CNN
 F 2 "" H 4700 2850 50  0000 C CNN
@@
 	5050 4400 5050 4500
 Connection ~ 5050 4500
+$Comp
+L LM358 U6
+U 1 1 586DE744
+P 5550 3200
+F 0 "U6" H 5550 3400 50  0000 L CNN
+F 1 "LM358" H 5550 3000 50  0000 L CNN
+F 2 "Housings_DIP:DIP-8_W7.62mm_LongPads" H 5550 3200 50  0001 C CNN
+F 3 "" H 5550 3200 50  0000 C CNN
+	1    5550 3200
+	-1   0    0    1
+$EndComp
+$Comp
+L LM358 U6
+U 2 1 586DE78F
+P 5550 4500
+F 0 "U6" H 5550 4700 50  0000 L CNN
+F 1 "LM358" H 5550 4300 50  0000 L CNN
+F 2 "Housings_DIP:DIP-8_W7.62mm_LongPads" H 5550 4500 50  0001 C CNN
+F 3 "" H 5550 4500 50  0000 C CNN
+	2    5550 4500
+	-1   0    0    1
+$EndComp
 $EndSCHEMATC

Commit message: a
Parts:
- removed R22, R23: 10k, Resistors_SMD:R_0805_HandSoldering, symbol R
- added RV2: 20k, Potentiometers:Potentiometer_Triwood_RM-065, symbol POT-RESCUE-v2
Connections:
- net 12Vrelay: now also P15.1 (P1), U6.8 (V+), RV2.1; no longer P15.4 (P4), U6.8 (V+)
- net GND: now also P15.4 (P4), U6.4 (V-), RV2.3; no longer P15.1 (P1), U6.4 (V-)
- net off: now also P15.2 (P2), U6.7; no longer P15.3 (P3), U6.1
- net onFan: now also P15.3 (P3), U6.1; no longer P15.2 (P2), U6.7
- net at U6.3 (+): now also RV3.2
- net at U6.5 (+): now also RV2.2; no longer RV3.2
Other:
- moved on the sheet: U6A, U6B
Changed lines of the file:
@@
 $EndDescr
 $Comp
-L GND #PWR59
+L GND #PWR054
 U 1 1 5872C09D
 P 5650 4100
-F 0 "#PWR59" H 5650 3850 50  0001 C CNN
+F 0 "#PWR054" H 5650 3850 50  0001 C CNN
 F 1 "GND" H 5650 3950 50  0000 C CNN
 F 2 "" H 5650 4100 50  0000 C CNN
@@
 $EndComp
 $Comp
-L GND #PWR61
+L GND #PWR055
 U 1 1 5872C0AA
 P 6400 3750
-F 0 "#PWR61" H 6400 3500 50  0001 C CNN
+F 0 "#PWR055" H 6400 3500 50  0001 C CNN
 F 1 "GND" H 6400 3600 50  0000 C CNN
 F 2 "" H 6400 3750 50  0000 C CNN
@@
 Text Notes 6550 3650 0    60   ~ 0
 90*C-10k\nturn off relayN, relayS
-$Comp
-L R R22
-U 1 1 5872C0B2
-P 6100 2900
-F 0 "R22" V 6180 2900 50  0000 C CNN
-F 1 "10k" V 6100 2900 50  0000 C CNN
-F 2 "Resistors_SMD:R_0805_HandSoldering" V 6030 2900 50  0001 C CNN
-F 3 "" H 6100 2900 50  0000 C CNN
-	1    6100 2900
-	-1   0    0    1
-$EndComp
-$Comp
-L R R23
-U 1 1 5872C0B9
-P 6100 3500
-F 0 "R23" V 6180 3500 50  0000 C CNN
-F 1 "10k" V 6100 3500 50  0000 C CNN
-F 2 "Resistors_SMD:R_0805_HandSoldering" V 6030 3500 50  0001 C CNN
-F 3 "" H 6100 3500 50  0000 C CNN
-	1    6100 3500
-	-1   0    0    1
-$EndComp
 $Comp
 L POT-RESCUE-v2 RV3
@@
 $EndComp
 $Comp
-L GND #PWR60
+L GND #PWR056
 U 1 1 5872C0C7
 P 6100 4850
-F 0 "#PWR60" H 6100 4600 50  0001 C CNN
+F 0 "#PWR056" H 6100 4600 50  0001 C CNN
 F 1 "GND" H 6100 4700 50  0000 C CNN
 F 2 "" H 6100 4850 50  0000 C CNN
@@
 Connection ~ 6400 3700
 Wire Wire Line
-	6100 3050 6100 3350
-Wire Wire Line
-	6100 3650 6100 3700
-Wire Wire Line
-	5850 3300 6100 3300
-Connection ~ 6100 3300
+	6100 3450 6100 3700
 Wire Wire Line
 	5850 4400 5950 4400
@@
 	6100 4750 6100 4850
 Wire Wire Line
-	6100 2550 6100 2750
+	6100 2550 6100 3150
 Wire Wire Line
 	6100 4450 6100 4400
@@
 F 3 "" H 4850 2500 50  0000 C CNN
 	1    4850 2500
-	0    -1   -1   0
-$EndComp
-$Comp
-L GND #PWR58
+	0    1    -1   0
+$EndComp
+$Comp
+L GND #PWR057
 U 1 1 5872CED6
 P 4700 2850
-F 0 "#PWR58" H 4700 2600 50  0001 C CNN
+F 0 "#PWR057" H 4700 2600 50  0001 C CNN
 F 1 "GND" H 4700 2700 50  0000 C CNN
 F 2 "" H 4700 2850 50  0000 C CNN
@@
 L LM358 U6
 U 1 1 586DE744
+P 5550 4500
+F 0 "U6" H 5550 4700 50  0000 L CNN
+F 1 "LM358" H 5550 4300 50  0000 L CNN
+F 2 "Housings_DIP:DIP-8_W7.62mm_LongPads" H 5550 4500 50  0001 C CNN
+F 3 "" H 5550 4500 50  0000 C CNN
+	1    5550 4500
+	-1   0    0    1
+$EndComp
+$Comp
+L LM358 U6
+U 2 1 586DE78F
 P 5550 3200
 F 0 "U6" H 5550 3400 50  0000 L CNN
@@
 F 2 "Housings_DIP:DIP-8_W7.62mm_LongPads" H 5550 3200 50  0001 C CNN
 F 3 "" H 5550 3200 50  0000 C CNN
-	1    5550 3200
+	2    5550 3200
 	-1   0    0    1
 $EndComp
 $Comp
-L LM358 U6
-U 2 1 586DE78F
-P 5550 4500
-F 0 "U6" H 5550 4700 50  0000 L CNN
-F 1 "LM358" H 5550 4300 50  0000 L CNN
-F 2 "Housings_DIP:DIP-8_W7.62mm_LongPads" H 5550 4500 50  0001 C CNN
-F 3 "" H 5550 4500 50  0000 C CNN
-	2    5550 4500
-	-1   0    0    1
-$EndComp
+L POT-RESCUE-v2 RV2
+U 1 1 58763EA0
+P 6100 3300
+F 0 "RV2" H 6100 3220 50  0000 C CNN
+F 1 "20k" H 6100 3300 50  0000 C CNN
+F 2 "Potentiometers:Potentiometer_Triwood_RM-065" H 6100 3300 50  0001 C CNN
+F 3 "" H 6100 3300 50  0000 C CNN
+	1    6100 3300
+	0    -1   1    0
+$EndComp
+Wire Wire Line
+	5950 3300 5850 3300
 $EndSCHEMATC
