File: project/load_v3/v3.kicad_pcb (KiCad board)
At the start: 2 copper layers, 150.5 x 90.8 mm, 118 parts, among them IC1 ATMEGA328-P, P1 12VAC, P10 relay, P2 NGUON, P3 SAC, P4 12N60C, P5 CONN_01X02, P6 button, P7 UART, P8 FAN, P9 7-seg, Q1 Q_NPN_BCE, Q2 Q_NPN_BCE, Q3 Q_NPN_BCE, SW1 reset, U1 LM7812CT, U2 LM7805CT, U3 ICL7660, U4 TL431, U5 LM324N, U6 LM324N, U7 LM7812CT, Y1 16MHz

Commit message: a
Parts:
- removed C18: 100nF, Capacitors_THT:C_Rect_L7_W2_P5
- removed C19: 22nF, Capacitors_THT:C_Disc_D3_P2.5
- removed C21: 100nF, Capacitors_THT:C_Disc_D3_P2.5
- removed R46: 10k, Resistors_THT:Resistor_Horizontal_RM7mm
- removed R47, R48, R49, R50, R51, R52, R53, R54, R55, R56, R57: 0R, Wire_Connections_Bridges:WireConnection_0.80mmDrill
- removed RV2: 20k, Potentiometers:Potentiometer_Bourns_3296W_3-8Zoll_Inline_ScrewUp
- removed U6: LM324N, Housings_DIP:DIP-14_W7.62mm_LongPads
- added C14: 22nF, Capacitors_THT:C_Disc_D3_P2.5, F.Cu at (153.0, 273.1)
- added C8: 22nF, Capacitors_THT:C_Disc_D3_P2.5, F.Cu at (138.4, 273.7)
- added D12: 4001, Diodes_THT:Diode_DO-35_SOD27_Horizontal_RM10, F.Cu at (128.1, 98.7)
- added D13: 4001, Diodes_THT:Diode_DO-35_SOD27_Horizontal_RM10, F.Cu at (89.9, 142.4)
- added D14: Led_Small, LEDs:LED-3MM, F.Cu at (207.4, 102.9)
- added P11: G, Connectors:XH2.54-3P, F.Cu at (203.2, 64.9)
- added P12: N, Connectors_Phoenix:PhoenixContact_MCV-G_02x5.08mm_Vertical, F.Cu at (104.4, 135.0)
- added P13: S, Connectors_Phoenix:PhoenixContact_MCV-G_02x5.08mm_Vertical, F.Cu at (130.3, 108.9)
- added P14: pwr, Connectors_Phoenix:PhoenixContact_MCV-G_02x5.08mm_Vertical, F.Cu at (97.2, 268.0)
- added P15: overheat, Connectors:XH2.54-4P, F.Cu at (316.2, 68.0)
- added P16: g, Connectors:XH2.54-3P, F.Cu at (203.2, 276.2)
- added Q4: 2n222, TO_SOT_Packages_THT:TO-92_Molded_Wide_Oval_Reverse, F.Cu at (153.5, 109.2)
- added Q5: 2n222, TO_SOT_Packages_THT:TO-92_Molded_Wide_Oval_Reverse, F.Cu at (139.2, 122.3)
- added Q6: Q_NMOS_GDS, TO_SOT_Packages_THT:TO-247_Vertical_Neutral123, F.Cu at (118.7, 264.8)
- added Q7: Q_NMOS_GDS, TO_SOT_Packages_THT:TO-247_Vertical_Neutral123, F.Cu at (163.2, 264.8)
- added R58: 470R, Resistors_THT:Resistor_Horizontal_RM7mm, F.Cu at (113.0, 271.1)
- added R59: 1k, Resistors_THT:Resistor_Horizontal_RM7mm, F.Cu at (128.9, 279.4)
- added R60: 0.5R, Resistors_THT:Resistor_Vertical_RM7.5mm, F.Cu at (133.3, 272.4)
- added R61: 470R, Resistors_THT:Resistor_Horizontal_RM7mm, F.Cu at (152.4, 264.8)
- added R62: 1k, Resistors_THT:Resistor_Horizontal_RM7mm, F.Cu at (168.9, 273.7)
- added R64: 0.5R, Resistors_THT:Resistor_Vertical_RM7.5mm, F.Cu at (177.2, 272.4)
- added RL1: onN, Relays_THT:Relay_SPDT_OMRON-G5Q, F.Cu at (107.1, 105.4)
- added RL2: onS, Relays_THT:Relay_SPDT_OMRON-G5Q, F.Cu at (89.3, 89.8)
- added RV3: 20k, Potentiometers:Potentiometer_Triwood_RM-065, F.Cu at (310.4, 74.6)
- added TH2: Thermistor, Discret:R3, F.Cu at (312.3, 82.1)
- added U8: LM358, Housings_DIP:DIP-8_W7.62mm_LongPads, F.Cu at (142.2, 270.5)
- added U9: LM324N, Housings_DIP:DIP-14_W7.62mm_LongPads, F.Cu at (298.4, 69.7)
- added VR3: 14D180V, Varistors:RV_Disc_D15.5_W3.9_P7.5, F.Cu at (91.6, 97.2)
- C1: footprint Capacitors_THT:C_Radial_D5_L6_P2.5 -> Capacitors_THT:C_Radial_D8_L11.5_P3.5
- C10, C12, C13, C9, R10, R11, R12, R13, R14, R15, R16, R17, R18, R2, R3, R9: moved to F.Cu
- D1: footprint Diodes_THT:Diode_Bridge_18.5x5.5 -> Diodes_THT:Diode_Bridge_KBP206
- D8: value 5.1V -> Led_Small; footprint Diodes_THT:Diode_DO-35_SOD27_Horizontal_RM10 -> LEDs:LED-3MM
- P10: value relay -> overheat
- P4: value 12N60C -> DS; footprint Connectors_Phoenix:PhoenixContact_MCV-G_05x5.08mm_Vertical -> Connectors_Phoenix:PhoenixContact_MCV-G_02x5.08mm_Vertical
- Q1, Q2, Q3, U4: footprint TO_SOT_Packages_THT:TO-92_Molded_Narrow -> TO_SOT_Packages_THT:TO-92_Molded_Wide_Oval_Reverse
- R22: value 470R -> 10k; footprint Resistors_THT:Resistor_Horizontal_RM7mm -> Resistors_SMD:R_0805_HandSoldering
- R23: value 1k -> 10k; footprint Resistors_THT:Resistor_Horizontal_RM7mm -> Resistors_SMD:R_0805_HandSoldering
- R28: value 330R -> 10k; footprint Resistors_THT:Resistor_Horizontal_RM7mm -> Resistors_SMD:R_0805_HandSoldering
- R29: footprint Resistors_THT:Resistor_Horizontal_RM15mm -> Resistors_THT:Resistor_Horizontal_RM7mm
- R30: value 180k -> 10k; footprint Resistors_THT:Resistor_Horizontal_RM15mm -> Resistors_THT:Resistor_Horizontal_RM7mm
- R41, R45: value 10k -> 470R; footprint Resistors_THT:Resistor_Horizontal_RM7mm -> Resistors_SMD:R_0805_HandSoldering
- VR1, VR2: value 14D470K -> 14D180V
- Y1: footprint Crystals:Crystal_HC52-U_Vertical -> Crystals:Crystal_HC50-U_Vertical
- moved R22 206.9 mm to (329.4, 66.6), turned to 0 degrees
- moved R23 190.2 mm to (315.8, 76.9), turned to 0 degrees
- moved R30 181.7 mm to (157.5, 277.5), turned to 90 degrees
- moved R28 169.9 mm to (319.6, 83.1)
- moved R29 162.1 mm to (124.5, 271.1)
- moved Q2 124.3 mm to (117.2, 145.0), turned to 0 degrees
- moved D1 123.6 mm to (86.9, 132.0), turned to 0 degrees
- moved R32 114.0 mm to (210.7, 75.1), turned to 0 degrees
- moved P8 113.5 mm to (235.4, 64.9), turned to 0 degrees
- moved HS2 113.3 mm to (88.7, 109.2), turned to 0 degrees
- moved R10 101.7 mm to (194.4, 64.4)
- moved C11 100.6 mm to (102.0, 152.2), turned to 0 degrees
- moved R42 100.1 mm to (146.4, 149.9), turned to 0 degrees
- moved IC1 96.7 mm to (77.9, 66.5), turned to 0 degrees
- moved P1 95.3 mm to (116.7, 126.3), turned to 0 degrees
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Connections:
- C10 pad 2: Net-(C10-Pad2) -> +5V
- C17 pad 2: Net-(C17-Pad2) -> G
- D7 pad 1: +12V -> 12Vrelay
- D8 pad 1: Net-(D8-Pad1) -> N-
- D8 pad 2: N- -> Net-(D8-Pad2)
- IC1 pad 25: senUN -> (no net)
- IC1 pad 27: Net-(IC1-Pad27) -> ok
- IC1 pad 28: Net-(IC1-Pad28) -> fail
- IC1 pad 7: Net-(C10-Pad2) -> +5V
- P10 pad 1: 12Vrelay -> N-
- P10 pad 2: onN -> onFan
- P10 pad 3: onS -> off
- P10 pad 4: N- -> 12Vrelay
- P6 pad 8: Net-(P6-Pad8) -> (no net)
- P8 pad 1: +12V -> 12Vrelay
- P9 pad 4: Net-(P9-Pad4) -> (no net)
- Q3 pad 3: Net-(Q3-Pad3) -> N-
- R1 pad 2: 12V2 -> (no net)
- R21 pad 1: Net-(C17-Pad2) -> G
- R22 pad 1: G -> Net-(R22-Pad1)
- R22 pad 2: Net-(C19-Pad2) -> 12Vrelay
- R23 pad 1: Net-(R23-Pad1) -> N-
- R23 pad 2: Net-(C19-Pad1) -> Net-(R22-Pad1)
- R26 pad 1: Net-(R23-Pad1) -> S
- R28 pad 1: Net-(D8-Pad1) -> Net-(R28-Pad1)
- R28 pad 2: senUN -> 12Vrelay
- R29 pad 1: Net-(R29-Pad1) -> Net-(Q6-Pad3)
- R29 pad 2: N- -> Net-(Q6-Pad1)
- R30 pad 1: N+ -> Net-(Q7-Pad3)
- R30 pad 2: Net-(R29-Pad1) -> Net-(Q7-Pad1)
- R40 pad 1: Net-(R40-Pad1) -> Net-(Q1-Pad1)
- R40 pad 2: Net-(R40-Pad2) -> off
- R41 pad 1: THa -> Net-(D8-Pad2)
- R41 pad 2: +12V -> ok
- R44 pad 1: Net-(R44-Pad1) -> Net-(Q3-Pad1)
- R44 pad 2: Net-(Q3-Pad1) -> onFan
- R45 pad 2: +12V -> fail
- R7 pad 1: Net-(C10-Pad2) -> +5V
- U3 pad 1: Net-(U3-Pad1) -> (no net)
- U3 pad 6: Net-(U3-Pad6) -> (no net)
- U3 pad 7: Net-(U3-Pad7) -> (no net)
- U3 pad 8: Net-(R53-Pad2) -> +5V
- U5 pad 1: Net-(D11-Pad1) -> Net-(D10-Pad1)
- U5 pad 10: Net-(R26-Pad2) -> Net-(R32-Pad1)
- U5 pad 11: -5V -> (no net)
- U5 pad 12: Net-(C17-Pad2) -> Net-(R26-Pad2)
- U5 pad 13: Net-(C19-Pad1) -> Net-(R25-Pad1)
- U5 pad 14: Net-(C19-Pad2) -> Net-(D9-Pad1)
- U5 pad 2: Net-(D11-Pad1) -> Net-(R38-Pad2)
- U5 pad 3: Net-(R32-Pad1) -> Net-(R37-Pad1)
- U5 pad 4: 12V2 -> (no net)
- U5 pad 5: Net-(R29-Pad1) -> N-
- U5 pad 6: Net-(D8-Pad1) -> Net-(R34-Pad1)
- U5 pad 7: Net-(D8-Pad1) -> Net-(R34-Pad2)
- U5 pad 8: Net-(D9-Pad1) -> Net-(D11-Pad1)
- U5 pad 9: Net-(R25-Pad1) -> Net-(D11-Pad1)
Routing:
- net N-: track 701.6 -> 0.00 mm
- net (no net): track 482.6 -> 0.00 mm
- net +12V: track 137.4 -> 0.00 mm
- net THa: track 113.7 -> 0.00 mm
- net +5V: track 109.1 -> 0.00 mm
- net S-: track 105.1 -> 0.00 mm
- net G: track 101.6 -> 0.00 mm
- net 17V: track 94.6 -> 0.00 mm
- net Net-(R32-Pad1): track 76.0 -> 0.00 mm
- net Net-(R23-Pad1): track 65.4 -> 0.00 mm
- net Net-(R52-Pad2): track 57.6 -> 0.00 mm
- net S: track 54.7 -> 0.00 mm
- net -5V: track 45.0 -> 0.00 mm
- net Net-(R40-Pad1): track 43.2 -> 0.00 mm
- net Net-(Q3-Pad3): track 42.7 -> 0.00 mm
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- removed copper zone on B.Cu, net N-
Other:
- board outline removed
- net class +12V removed
- net class +5V removed
- net class Default: clearance 0.25 -> 0.2
- rule pad_to_mask_clearance: 0.2 -> 0
- rule trace_clearance: 0.25 -> 0.2
- rule trace_min: 0.25 -> 0.2

Commit message: a
Parts:
- removed P12: N, Connectors_Phoenix:PhoenixContact_MCV-G_02x5.08mm_Vertical
- removed P13: S, Connectors_Phoenix:PhoenixContact_MCV-G_02x5.08mm_Vertical
- removed U9: LM324N, Housings_DIP:DIP-14_W7.62mm_LongPads
- added U6: LM358, Housings_DIP:DIP-8_W7.62mm_LongPads, F.Cu at (153.0, 257.2)
- C10, C12, C13, C9, R10, R11, R12, R13, R14, R15, R16, R17, R18, R2, R22, R23, R28, R3, R41, R45, R9: moved to B.Cu
- RL1, RL2: footprint Relays_THT:Relay_SPDT_OMRON-G5Q -> Relays_THT:Relay_SANYOU_SRD_Series_Form_C
- moved R14 471.7 mm to (611.5, 176.5)
- moved R16 466.6 mm to (593.7, 177.2)
- moved R12 457.8 mm to (574.7, 174.6)
- moved R13 445.3 mm to (551.2, 174.6)
- moved R45 442.1 mm to (626.1, 135.9)
- moved R3 438.5 mm to (640.1, 135.9)
- moved R18 438.1 mm to (532.1, 173.4)
- moved R10 437.3 mm to (613.4, 189.9)
- moved R41 436.5 mm to (615.3, 149.9)
- moved C10 436.4 mm to (629.9, 148.0)
- moved R2 436.0 mm to (648.3, 152.4)
- moved C9 434.4 mm to (654.7, 142.9)
- moved R9 429.0 mm to (592.5, 191.8)
- moved R17 418.1 mm to (573.4, 190.5)
- moved D6 412.7 mm to (645.2, 54.6)
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Connections:
- D5 pad 2: N+ -> rN+
- P3 pad 2: D -> S+
- RL1 pad 1: Net-(D12-Pad2) -> N+
- RL1 pad 2: Net-(P12-Pad2) -> Net-(D12-Pad2)
- RL1 pad 3: Net-(P12-Pad1) -> rN+
- RL2 pad 1: Net-(D13-Pad2) -> D
- RL2 pad 2: Net-(P13-Pad2) -> Net-(D13-Pad2)
- RL2 pad 3: Net-(P13-Pad1) -> S+
Routing:
- net S: track 0.00 -> 109.3 mm
- net D: track 0.00 -> 97.0 mm
- net G: track 0.00 -> 61.5 mm
- net -5V: track 0.00 -> 61.4 mm
- net +12V: track 0.00 -> 56.4 mm
- net 12Vrelay: track 0.00 -> 35.2 mm
- net Net-(C8-Pad1): track 0.00 -> 33.5 mm
- net Net-(R28-Pad1): track 0.00 -> 29.0 mm
- net Net-(Q6-Pad3): track 0.00 -> 22.8 mm
- net Net-(C14-Pad2): track 0.00 -> 22.1 mm
- net N-: track 0.00 -> 21.0 mm
- net Net-(C8-Pad2): track 0.00 -> 18.8 mm
- net Net-(Q7-Pad3): track 0.00 -> 18.5 mm
- net onFan: track 0.00 -> 15.4 mm
- net Net-(C14-Pad1): track 0.00 -> 10.7 mm
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Other:
- board outline added: 148.9 x 22.9 mm
- net class Default: clearance 0.2 -> 0.25
- rule trace_clearance: 0.2 -> 0.25

Commit message: a
Parts:
- added P12: opto, Connectors:XH2.54-4P, F.Cu at (327.0, -15.2)
- added R46: 10k, Resistors_THT:Resistor_Horizontal_RM7mm, F.Cu at (290.2, 50.8)
- added U10: PC817, Housings_DIP:DIP-4_W7.62mm_LongPads, F.Cu at (315.0, -16.5)
- added U9: PC817, Housings_DIP:DIP-4_W7.62mm_LongPads, F.Cu at (315.0, -24.1)
- R42: value 1k -> 10k
- moved R42 280.8 mm to (290.2, 47.6), turned to 180 degrees
Connections:
- D6 pad 1: led -> N-
- IC1 pad 13: led -> Net-(IC1-Pad13)
- IC1 pad 14: Net-(IC1-Pad14) -> start
- Q2 pad 2: onS -> onN
- Q5 pad 1: onS -> onN
- R19 pad 1: +5V -> start
- R42 pad 1: onN -> opto_start
- R42 pad 2: Net-(IC1-Pad14) -> start
- R43 pad 1: onS -> onN

Commit message: a
Parts:
- removed D6: Led_Small, LEDs:LED-3MM
- removed VR2: 14D180V, Varistors:RV_Disc_D15.5_W3.9_P7.5
- added D15: Led_Small, LEDs:LED-3MM, F.Cu at (189.0, 161.8)
- added D16: Led_Small, LEDs:LED-3MM, F.Cu at (189.0, 157.4)
- added P13: tac_auto, Connectors:XH2.54-2P, F.Cu at (194.6, 184.2)
- added R47: 470R, Resistors_SMD:R_0805_HandSoldering, B.Cu at (180.1, 162.9)
- R19: footprint Resistors_THT:Resistor_Horizontal_RM7mm -> Resistors_SMD:R_0805_HandSoldering; moved to B.Cu
- R42, R46: value 10k -> 1k
- moved P8 609.6 mm to (49.3, 163.8), turned to 270 degrees
- moved R40 587.7 mm to (60.5, 186.7), turned to 90 degrees
- moved R32 569.0 mm to (67.1, 179.1), turned to 270 degrees
- moved D4 560.4 mm to (76.1, 174.0), turned to 90 degrees
- moved C15 552.8 mm to (106.1, 227.1), turned to 180 degrees
- moved Q3 548.9 mm to (54.9, 167.6), turned to 90 degrees
- moved R6 547.7 mm to (76.1, 168.5), turned to 90 degrees
- moved C7 543.5 mm to (84.9, 173.0)
- moved D7 529.2 mm to (47.8, 160.3)
- moved R21 522.0 mm to (90.2, 169.9), turned to 270 degrees
- moved R26 515.9 mm to (92.1, 189.2), turned to 90 degrees
- moved R10 515.1 mm to (98.4, 200.7)
- moved D14 510.3 mm to (125.7, 213.0)
- moved R34 507.6 mm to (121.2, 194.6)
- moved C16 507.5 mm to (96.7, 167.1), turned to 180 degrees
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Connections:
- IC1 pad 13: Net-(IC1-Pad13) -> l_auto
- IC1 pad 14: start -> l_start
- R19 pad 1: start -> Net-(D15-Pad2)
- R19 pad 2: Net-(D6-Pad2) -> l_auto
- R42 pad 2: start -> l_start
- R46 pad 2: Net-(IC1-Pad13) -> l_auto
- U10 pad 1: opto_start -> opto_auto
- U5 pad 1: Net-(D10-Pad1) -> Net-(D9-Pad1)
- U5 pad 10: Net-(R32-Pad1) -> Net-(R37-Pad1)
- U5 pad 12: Net-(R26-Pad2) -> Net-(R32-Pad1)
- U5 pad 13: Net-(R25-Pad1) -> Net-(D11-Pad1)
- U5 pad 14: Net-(D9-Pad1) -> Net-(D11-Pad1)
- U5 pad 2: Net-(R38-Pad2) -> Net-(R25-Pad1)
- U5 pad 3: Net-(R37-Pad1) -> Net-(R26-Pad2)
- U5 pad 8: Net-(D11-Pad1) -> Net-(D10-Pad1)
- U5 pad 9: Net-(D11-Pad1) -> Net-(R38-Pad2)
- U9 pad 1: opto_auto -> opto_start
- VR1 pad 2: S- -> N-
Routing:
- net N-: track 21.0 -> 252.8 mm
- net Net-(Q1-Pad1): track 0.00 -> 127.7 mm
- net S-: track 0.00 -> 106.6 mm
- net S: track 109.3 -> 197.5 mm
- net 12Vrelay: track 35.2 -> 117.6 mm, vias 0 -> 4
- net onN: track 0.00 -> 57.0 mm, vias 0 -> 2
- net D: track 97.0 -> 135.9 mm
- net N+: track 0.00 -> 23.5 mm
- net S+: track 0.00 -> 11.9 mm
- net Net-(D12-Pad2): track 0.00 -> 11.8 mm
- net Net-(D13-Pad2): track 0.00 -> 11.7 mm
- net rN+: track 0.00 -> 7.52 mm

Commit message: a
Parts:
- moved R18 9.89 mm to (106.0, 199.4)
- moved R9 9.44 mm to (92.1, 199.4)
- moved R17 8.39 mm to (106.0, 205.1)
- moved R16 7.84 mm to (106.0, 210.8)
- moved R10 7.75 mm to (92.1, 205.1)
- moved R14 7.36 mm to (106.0, 222.2)
- moved R15 7.36 mm to (106.0, 216.5)
- moved R11 6.84 mm to (92.1, 210.8)
- moved R13 6.84 mm to (92.1, 222.2)
- moved R12 6.35 mm to (92.1, 216.5)
- moved C15 1.69 mm to (105.4, 228.6), turned to 90 degrees
- moved D5 1.49 mm to (69.3, 206.2)
- moved VR1 0.80 mm to (72.1, 206.2)
- moved U7 0.57 mm to (114.3, 227.3)
- moved P2 0.51 mm to (48.4, 219.7)
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Routing:
- net N-: track 252.8 -> 171.8 mm
- net 12Vrelay: track 117.6 -> 59.7 mm, vias 4 -> 0
- net onN: track 57.0 -> 38.1 mm, vias 2 -> 0
- net S: track 197.5 -> 181.6 mm
- net S-: track 106.6 -> 95.8 mm
- net Net-(Q1-Pad1): track 127.7 -> 119.8 mm
- net rN+: track 7.52 -> 8.91 mm
- net N+: track 23.5 -> 24.5 mm
- net D: track 135.9 -> 136.8 mm
Other:
- board size 148.9 x 22.9 mm -> 183.7 x 123.1 mm
- net class Default: clearance 0.25 -> 0.35
- rule trace_clearance: 0.25 -> 0.35

Commit message: a
Parts:
- R4: footprint Resistors_THT:Resistor_Horizontal_RM7mm -> Resistors_SMD:R_0805_HandSoldering; moved to B.Cu
- moved P14 217.6 mm to (111.0, 68.1), turned to 180 degrees
- moved R58 192.5 mm to (105.4, 89.4), turned to 270 degrees
- moved Q6 181.0 mm to (112.9, 95.0), turned to 270 degrees
- moved R29 180.9 mm to (108.5, 97.0), turned to 90 degrees
- moved R59 176.3 mm to (108.5, 100.6), turned to 270 degrees
- moved R60 159.6 mm to (107.2, 114.6), turned to 180 degrees
- moved C8 146.8 mm to (113.5, 121.4), turned to 180 degrees
- moved U8 143.0 mm to (113.5, 124.5), turned to 270 degrees
- moved TH2 140.9 mm to (37.8, 200.8), turned to 0 degrees
- moved C14 131.9 mm to (111.0, 135.1), turned to 180 degrees
- moved RV3 128.8 mm to (40.4, 208.4), turned to 90 degrees
- moved R23 126.8 mm to (39.1, 213.4), turned to 270 degrees
- moved R28 123.0 mm to (39.1, 218.6), turned to 270 degrees
- moved R61 117.8 mm to (108.5, 149.4), turned to 90 degrees
- moved U6 117.5 mm to (41.7, 219.8), turned to 180 degrees
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Connections:
- P1 pad 1: Net-(D1-Pad2) -> Net-(D1-Pad4)
- P1 pad 2: Net-(D1-Pad4) -> Net-(D1-Pad2)
- U5 pad 11: (no net) -> -5V
- U5 pad 4: (no net) -> +12V
Routing:
- net N-: track 171.8 -> 496.7 mm
- net 12Vrelay: track 59.7 -> 177.5 mm, vias 0 -> 2
- net 17V: track 0.00 -> 99.1 mm
- net +12V: track 56.4 -> 144.0 mm
- net Net-(R32-Pad1): track 0.00 -> 78.2 mm
- net Net-(R26-Pad2): track 0.00 -> 46.3 mm
- net +5V: track 0.00 -> 35.9 mm
- net Net-(D10-Pad1): track 0.00 -> 28.8 mm
- net onN: track 38.1 -> 57.1 mm, vias 0 -> 2
- net Net-(D1-Pad2): track 0.00 -> 18.1 mm
- net Net-(R34-Pad1): track 0.00 -> 14.7 mm
- net Net-(D9-Pad1): track 0.00 -> 13.5 mm
- net senIS: track 0.00 -> 13.4 mm
- net D: track 136.8 -> 149.9 mm
- net senUS: track 0.00 -> 13.1 mm
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Other:
- board size 183.7 x 123.1 mm -> 180 x 201.4 mm

Commit message: a
Parts:
- removed R22, R23: 10k, Resistors_SMD:R_0805_HandSoldering
- added RV2: 20k, Potentiometers:Potentiometer_Triwood_RM-065, F.Cu at (181.8, 53.0)
- R5: footprint Resistors_THT:Resistor_Horizontal_RM7mm -> Resistors_SMD:R_0805_HandSoldering; moved to B.Cu
- moved U6 227.2 mm to (198.8, 55.8), turned to 270 degrees
- moved R28 222.9 mm to (196.3, 60.6), turned to 0 degrees
- moved P15 216.7 mm to (204.1, 62.6), turned to 90 degrees
- moved TH2 213.3 mm to (192.4, 53.7), turned to 180 degrees
- moved RV3 205.0 mm to (186.8, 64.9)
- moved D3 143.4 mm to (195.7, 118.5), turned to 180 degrees
- moved P13 140.3 mm to (207.3, 100.1), turned to 90 degrees
- moved R5 136.6 mm to (191.8, 120.8), turned to 0 degrees
- moved D10 136.4 mm to (164.1, 109.1), turned to 0 degrees
- moved C22 136.4 mm to (169.2, 96.1)
- moved R31 136.4 mm to (164.1, 93.5)
- moved R41 136.4 mm to (186.0, 109.5), turned to 0 degrees
- moved P10 135.2 mm to (68.7, 77.6)
- moved R25 134.7 mm to (143.1, 96.5)
- moved R44 133.8 mm to (72.8, 77.6)
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Connections:
- IC1 pad 23: senIN -> senUS
- IC1 pad 24: senUS -> senIN
- IC1 pad 25: (no net) -> senIS
- IC1 pad 26: senIS -> (no net)
- P15 pad 1: N- -> 12Vrelay
- P15 pad 2: onFan -> off
- P15 pad 3: off -> onFan
- P15 pad 4: 12Vrelay -> N-
- P16 pad 1: -5V -> +12V
- P16 pad 3: +12V -> -5V
- R1 pad 2: (no net) -> +12V
- R36 pad 2: senIS -> (no net)
- U6 pad 1: off -> onFan
- U6 pad 3: Net-(R22-Pad1) -> Net-(RV3-Pad2)
- U6 pad 5: Net-(RV3-Pad2) -> Net-(RV2-Pad2)
- U6 pad 7: onFan -> off
Routing:
- net N-: track 496.7 -> 958.0 mm, vias 0 -> 2
- net +12V: track 144.0 -> 272.3 mm, vias 0 -> 4
- net -5V: track 61.4 -> 179.6 mm, vias 0 -> 2
- net 12Vrelay: track 177.5 -> 274.9 mm
- net Net-(IC1-Pad15): track 0.00 -> 89.5 mm
- net l_start: track 0.00 -> 64.7 mm
- net +5V: track 35.9 -> 99.7 mm
- net l_auto: track 0.00 -> 58.4 mm
- net pwm: track 0.00 -> 55.3 mm
- net Net-(R32-Pad1): track 78.2 -> 110.2 mm
- net Net-(RV2-Pad2): track 0.00 -> 25.9 mm
- net Net-(P12-Pad4): track 0.00 -> 25.8 mm
- net Net-(C16-Pad2): track 0.00 -> 25.7 mm
- net Net-(D9-Pad1): track 13.5 -> 39.0 mm
- net Net-(P12-Pad3): track 0.00 -> 23.8 mm
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- added copper zone on B.Cu, net (none)
- added copper zone on B.Cu, net N-
Other:
- board size 180 x 201.4 mm -> 152.4 x 86.4 mm
